Commit message: test

File: odrive_botwheel_explorer/description/urdf/diffbot.ros2_control.xacro (robot description, xacro)
@@ -19,5 +19,5 @@
       </joint>
       <joint name="${prefix}right_wheel_joint">
-        <param name="node_id">1</param>
+        <param name="node_id">0</param>
       </joint>
     </ros2_control>

File: odrive_botwheel_explorer/description/urdf/diffbot_description.urdf.xacro (robot description, xacro)
@@ -10,5 +10,5 @@
   <xacro:property name="wheel_mass" value="0.3" /> <!-- arbitrary value for wheel mass -->
   <xacro:property name="wheel_len" value="0.020" />
-  <xacro:property name="wheel_radius" value="0.015" />
+  <xacro:property name="wheel_radius" value="0.00015" />
   <xacro:property name="caster_wheel_mass" value="0.1" /> <!-- arbitrary value for caster wheel mass -->
   <xacro:property name="caster_wheel_radius" value="0.015" />
